File: mouse-joystick-pcb/motor-0.kicad_sch (KiCad schematic)
At the start: 24 parts, among them J1 Molex_Pico-Clasp_Horizontal, U1 MAX6816, U401 TMC5130A-TA, X401 16MHz

Commit message: Make schematic changes
Parts:
- removed X401: 16MHz, Janelia:OSC_ECS-2520S33-160-FN-TR, symbol Janelia:Oscillator_16MHz_ECS-2520S33
Changed lines of the file:
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@@
-    )
-  )
-  (symbol (lib_id "Janelia:Oscillator_16MHz_ECS-2520S33") (at 71.12 40.64 0) (unit 1)
-    (in_bom yes) (on_board yes) (dnp no)
-    (property "Reference" "X401" (at 76.2 34.29 0)
-      (effects (font (size 1.27 1.27)) (justify left))
-    )
-    (property "Value" "16MHz" (at 72.39 46.99 0)
-      (effects (font (size 1.27 1.27)) (justify left))
-    )
-    (property "Footprint" "Janelia:OSC_ECS-2520S33-160-FN-TR" (at 82.55 49.53 0)
-      (effects (font (size 1.27 1.27)) hide)
-    )
-    (property "Datasheet" "" (at 66.675 37.465 0)
-      (effects (font (size 1.27 1.27)) hide)
-    )
-    (property "Manufacturer" "ECS Inc." (at 71.12 40.64 0)
-      (effects (font (size 1.27 1.27)) hide)
-    )
-    (property "Manufacturer Part Number" "ECS-2520S33-160-FN-TR" (at 71.12 40.64 0)
-      (effects (font (size 1.27 1.27)) hide)
-    )
-    (property "Vendor" "Digi-Key" (at 71.12 40.64 0)
-      (effects (font (size 1.27 1.27)) hide)
-    )
-    (property "Vendor Part Number" "XC2195CT-ND" (at 71.12 40.64 0)
-      (effects (font (size 1.27 1.27)) hide)
-    )
-    (property "Synopsis" "XTAL OSC XO 16.0000MHZ HCMOS SMD" (at 71.12 40.64 0)
-      (effects (font (size 1.27 1.27)) hide)
-    )
-    (property "LCSC" "C2451298" (at 71.12 40.64 0)
-      (effects (font (size 1.27 1.27)) hide)
-    )
-    (property "Package" "SMD2520-4P" (at 71.12 40.64 0)
-      (effects (font (size 1.27 1.27)) hide)
-    )
-    (pin "4")
-    (pin "3")
-    (pin "1")
-    (pin "2")
-    (instances
-      (project "mouse-joystick-pcb"
-        (path "/df2b2e89-e055-4140-95de-f1df723db034/843743ad-cb97-4017-b3d5-10e69a46da88"
-          (reference "X401") (unit 1)
-        )
-      )
     )
   )

Commit message: Add components
Parts:
- removed C2, C3: 47uF_50V, Janelia:CAP_EEE1HA470XP, symbol Janelia:CP_47uF_50V_6.3x7.7mm
- removed C401, C403, C404, C407, C410: 0.1uF_100V, Janelia:C_0402_1005Metric, symbol Janelia:C_0.1uF_100V_0402
- removed C402: 22nF_100V, Janelia:C_0603_1608Metric, symbol Janelia:C_22nF_100V_0603
- removed C405: 0.47uF_35V, Janelia:C_0402_1005Metric, symbol Janelia:C_0.47uF_35V_0402
- removed C406: 2.2uF_35V, Janelia:C_0402_1005Metric, symbol Janelia:C_2.2uF_35V_0402
- removed C408, C411: 2.2uF_100V, Janelia:C_0805_2012Metric, symbol Janelia:C_2.2uF_100V_0805
- removed C409, C412: 100uF_50V, Janelia:CAP_EEEHAH101UAP, symbol Janelia:CP_100uF_50V_8x10.2mm
- removed J1: Molex_Pico-Clasp_Horizontal, Janelia:Molex_Pico-Clasp-501568_1x02_P1mm_Horizontal, symbol Janelia:Conn_01x02_P1mm_Molex_Pico-Clasp-501330_Horizontal
- removed R401: 2.2, Janelia:R_0402_1005Metric, symbol Janelia:R_2.2_0402
- removed R402, R403: 0.12, Janelia:R_1206_3216Metric, symbol Janelia:R_0.12_750mW_1206_CS
- removed U401: TMC5130A-TA, Janelia:TQFP-48-1EP_7x7mm_P0.5mm_EP5x5mm_ThermalVias, symbol Janelia:TMC5130A-TA
- added C10, C11: 2.2uF_100V, Janelia:C_0805_2012Metric, symbol Janelia:C_2.2uF_100V_0805
- added C12, C13: 100uF_50V, Janelia:CAP_EEEHAH101UAP, symbol Janelia:CP_100uF_50V_8x10.2mm
- added C2, C4, C5, C8, C9: 0.1uF_100V, Janelia:C_0402_1005Metric, symbol Janelia:C_0.1uF_100V_0402
- added C3: 22nF_100V, Janelia:C_0603_1608Metric, symbol Janelia:C_22nF_100V_0603
- added C6: 0.47uF_35V, Janelia:C_0402_1005Metric, symbol Janelia:C_0.47uF_35V_0402
- added C7: 47uF_10V, Janelia:C_0805_2012Metric, symbol Janelia:C_47uF_10V_0805
- added J1: Conn_01x04_P3.5mm_TBH_Horizontal_Screw, Janelia:PhoenixContact_MC_1,5_4-G-3.5_1x04_P3.50mm_Horizontal_Screw, symbol Janelia:Conn_01x04_P3.5mm_TBH_Horizontal_Screw
- added J2: Conn_01x02_P3.5mm_TBH_Horizontal_Screw, Janelia:PhoenixContact_MC_1,5_2-G-3.5_1x02_P3.50mm_Horizontal_Screw, symbol Janelia:Conn_01x02_P3.5mm_TBH_Horizontal_Screw
- added J3: Conn_01x05_P3.5mm_TBH_Horizontal_Screw, Janelia:PhoenixContact_MC_1,5_5-G-3.5_1x05_P3.50mm_Horizontal_Screw, symbol Janelia:Conn_01x05_P3.5mm_TBH_Horizontal_Screw
- added R5: 10, Janelia:R_0402_1005Metric, symbol Janelia:R_10_62.5mW_0402
- added U1: TMC5130A-TA, Janelia:TQFP-48-1EP_7x7mm_P0.5mm_EP5x5mm_ThermalVias, symbol Janelia:TMC5130A-TA
- added X1: 16MHz_3.3V, Janelia:OSC_ECS-2520S33-160-FN-TR, symbol Janelia:Oscillator_16MHz_3.3V
- renumbered U1 to U2
Connections:
- net +5V: now also C6.1, R5.1, U1.34 (VCC), U1.39 (VSA)
- net 5VOUT: now also C7.1, R5.2, U1.33 (5VOUT)
- net BMA1: now also J1.4 (Pin_4), U1.46 (OA1)
- net BMA2: now also J1.3 (Pin_3), U1.42 (OA2)
- net BMB1: now also J1.2 (Pin_2), U1.15 (OB1)
- net BMB2: now also J1.1 (Pin_1), U1.19 (OB2)
- net BRA: now also U1.44 (BRA)
- net BRB: now also U1.17 (BRB)
- net CIPO: now also U1.7 (SDO_NAO_CFG0)
- net CLOCK: now also U1.2 (CLK), X1.3 (OUT)
- net COPI: now also U1.5 (SDI_NAI_CFG1)
- net CPI: now also C3.2, U1.37 (CPI)
- net CPO: now also C3.1, U1.35 (CP0)
- net GND: now also C10.2, C11.2, C12.2, C13.2, C2.2, C5.2, C6.2, C7.2, C8.2, C9.2, J2.1 (Pin_1), U1.1 (TST_MODE), U1.11 (SD_MODE), U1.13 (GNDP), U1.23 (ENCN_DCO), U1.24 (ENCB_DCEN_CFG4), U1.25 (ENCA_DCIN_CFG5), U1.29 (~{DRV_EN}_CFG6), U1.30 (AIN_IREF), U1.31 (NC), U1.32 (GNDA), U1.36 (NC), U1.48 (GNDP), U1.49 (EP), U1.6 (NC), U1.9 (REFR_DIR), X1.2 (GND)
- net REFL: now also J2.2 (Pin_2)
- net REFL_DEBOUNCED: now also U1.8 (REFL_STEP)
- net SCK: now also U1.4 (SCK_CFG2)
- net VCP: now also C4.2, U1.38 (VCP)
- net VM: now also C10.1, C11.1, C12.1, C13.1, C4.1, C8.1, C9.1, U1.21 (VS), U1.40 (VS)
- net ~{CS}: now also U1.3 (~{CS}_CFG3)
- net VIO renamed +3.3V
- net +3.3V: now also C2.1, C5.1, U1.10 (VCC_IO), U1.12 (SPI_MODE), X1.4 (VDD)
Other:
- note removed: "1.64 A RMS"
- moved on the sheet: C1, R1, R2, U2
