File: mouse-joystick-pcb/mouse-joystick-pcb.kicad_sch (KiCad schematic)
At the start: 0 parts

Commit message: Start wiring schematics
Other:
- removed sheet torque-sensor
- sheet audio ports: added +5V, AUDIO, GND; removed none
- sheet microcontroller ports: added +3.3V, GND, SCL, SDA; removed none
- sheet power ports: added +5V, GND, VBB; removed none
Changed lines of the file:
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@@
     (company "Peter Polidoro")
   )
+  (wire (pts (xy 96.52 86.36) (xy 93.98 86.36))
+    (stroke (width 0) (type default))
+  )
+  (wire (pts (xy 127 91.44) (xy 129.54 91.44))
+    (stroke (width 0) (type default))
+  )
+  (wire (pts (xy 127 54.61) (xy 129.54 54.61))
+    (stroke (width 0) (type default))
+  )
+  (wire (pts (xy 127 59.69) (xy 129.54 59.69))
+    (stroke (width 0) (type default))
+  )
+  (wire (pts (xy 96.52 68.58) (xy 93.98 68.58))
+    (stroke (width 0) (type default))
+  )
   (wire (pts (xy 69.85 54.61) (xy 72.39 54.61))
     (stroke (width 0) (type default))
   )
+  (wire (pts (xy 96.52 66.04) (xy 93.98 66.04))
+    (stroke (width 0) (type default))
+  )
+  (wire (pts (xy 127 96.52) (xy 129.54 96.52))
+    (stroke (width 0) (type default))
+  )
+  (wire (pts (xy 96.52 71.12) (xy 93.98 71.12))
+    (stroke (width 0) (type default))
+  )
+  (wire (pts (xy 40.64 66.04) (xy 43.18 66.04))
+    (stroke (width 0) (type default))
+  )
+  (wire (pts (xy 127 99.06) (xy 129.54 99.06))
+    (stroke (width 0) (type default))
+  )
+  (wire (pts (xy 127 93.98) (xy 129.54 93.98))
+    (stroke (width 0) (type default))
+  )
+  (wire (pts (xy 40.64 68.58) (xy 43.18 68.58))
+    (stroke (width 0) (type default))
+  )
+  (wire (pts (xy 127 62.23) (xy 129.54 62.23))
+    (stroke (width 0) (type default))
+  )
+  (wire (pts (xy 69.85 86.36) (xy 72.39 86.36))
+    (stroke (width 0) (type default))
+  )
+  (wire (pts (xy 127 57.15) (xy 129.54 57.15))
+    (stroke (width 0) (type default))
+  )
+  (label "+3.3V" (at 127 59.69 180) (fields_autoplaced)
+    (effects (font (size 1.27 1.27)) (justify right bottom))
+  )
+  (label "+3.3V" (at 96.52 86.36 0) (fields_autoplaced)
+    (effects (font (size 1.27 1.27)) (justify left bottom))
+  )
+  (label "+5V" (at 127 93.98 180) (fields_autoplaced)
+    (effects (font (size 1.27 1.27)) (justify right bottom))
+  )
+  (label "GND" (at 127 99.06 180) (fields_autoplaced)
+    (effects (font (size 1.27 1.27)) (justify right bottom))
+  )
+  (label "GND" (at 96.52 71.12 0) (fields_autoplaced)
+    (effects (font (size 1.27 1.27)) (justify left bottom))
+  )
   (label "GND" (at 69.85 54.61 180) (fields_autoplaced)
     (effects (font (size 1.27 1.27)) (justify right bottom))
   )
+  (label "GND" (at 127 62.23 180) (fields_autoplaced)
+    (effects (font (size 1.27 1.27)) (justify right bottom))
+  )
+  (label "+3.3V" (at 127 96.52 180) (fields_autoplaced)
+    (effects (font (size 1.27 1.27)) (justify right bottom))
+  )
+  (label "+5V" (at 127 57.15 180) (fields_autoplaced)
+    (effects (font (size 1.27 1.27)) (justify right bottom))
+  )
+  (label "VAA" (at 96.52 66.04 0) (fields_autoplaced)
+    (effects (font (size 1.27 1.27)) (justify left bottom))
+  )
+  (label "+5V" (at 96.52 68.58 0) (fields_autoplaced)
+    (effects (font (size 1.27 1.27)) (justify left bottom))
+  )
+  (label "+5V" (at 40.64 66.04 180) (fields_autoplaced)
+    (effects (font (size 1.27 1.27)) (justify right bottom))
+  )
+  (label "VAA" (at 127 91.44 180) (fields_autoplaced)
+    (effects (font (size 1.27 1.27)) (justify right bottom))
+  )
+  (label "GND" (at 40.64 68.58 180) (fields_autoplaced)
+    (effects (font (size 1.27 1.27)) (justify right bottom))
+  )
+  (label "VAA" (at 127 54.61 180) (fields_autoplaced)
+    (effects (font (size 1.27 1.27)) (justify right bottom))
+  )
+  (label "GND" (at 69.85 86.36 180) (fields_autoplaced)
+    (effects (font (size 1.27 1.27)) (justify right bottom))
+  )
   (sheet (at 72.39 52.07) (size 21.59 5.08) (fields_autoplaced)
     (stroke (width 0.1524) (type solid))
@@
     )
   )
-  (sheet (at 161.29 52.07) (size 24.13 15.24) (fields_autoplaced)
-    (stroke (width 0.1524) (type solid))
-    (fill (color 0 0 0 0.0000))
-    (property "Sheetname" "torque-sensor" (at 161.29 51.3584 0)
-      (effects (font (size 1.27 1.27)) (justify left bottom))
-    )
-    (property "Sheetfile" "torque-sensor.kicad_sch" (at 161.29 67.8946 0)
-      (effects (font (size 1.27 1.27)) (justify left top))
-    )
-    (instances
-      (project "mouse-joystick-pcb"
-        (path "/df2b2e89-e055-4140-95de-f1df723db034" (page "9"))
-      )
-    )
-  )
   (sheet (at 43.18 63.5) (size 15.24 10.16) (fields_autoplaced)
     (stroke (width 0.1524) (type solid))
@@
       (effects (font (size 1.27 1.27)) (justify left top))
     )
+    (pin "AUDIO" input (at 43.18 71.12 180)
+      (effects (font (size 1.27 1.27)) (justify left))
+    )
+    (pin "GND" passive (at 43.18 68.58 180)
+      (effects (font (size 1.27 1.27)) (justify left))
+    )
+    (pin "+5V" passive (at 43.18 66.04 180)
+      (effects (font (size 1.27 1.27)) (justify left))
+    )
     (instances
       (project "mouse-joystick-pcb"
@@
       (effects (font (size 1.27 1.27)) (justify left top))
     )
+    (pin "SDA" bidirectional (at 93.98 90.17 0)
+      (effects (font (size 1.27 1.27)) (justify right))
+    )
+    (pin "SCL" output (at 93.98 92.71 0)
+      (effects (font (size 1.27 1.27)) (justify right))
+    )
+    (pin "GND" passive (at 72.39 86.36 180)
+      (effects (font (size 1.27 1.27)) (justify left))
+    )
+    (pin "+3.3V" passive (at 93.98 86.36 0)
+      (effects (font (size 1.27 1.27)) (justify right))
+    )
     (instances
       (project "mouse-joystick-pcb"
@@
       (effects (font (size 1.27 1.27)) (justify left top))
     )
-    (instances
+    (pin "VBB" passive (at 93.98 66.04 0)
+      (effects (font (size 1.27 1.27)) (justify right))
+    )
+    (pin "+5V" passive (at 93.98 68.58 0)
+      (effects (font (size 1.27 1.27)) (justify right))
+    )
+    (pin "GND" passive (at 93.98 71.12 0)
+      (effects (font (size 1.27 1.27)) (justify right))
+    )
+    (instances

Commit message: Finish v1.0 schematic
Other:
- sheet brake ports: added BRAKE_PWM, GND, VS; removed none
- sheet microcontroller ports: added AUDIO, BRAKE_PWM, CIPO, COPI, MOTOR_DIAG0_0, MOTOR_DIAG0_1, SCK, ~{MOTOR_CS_0}, ~{MOTOR_CS_1}; removed SCL, SDA
- sheet motor-0 ports: added DIAG0, VIO; removed +3.3V, ENABLE
- sheet motor-1 ports: added DIAG0, VIO; removed +3.3V, ENABLE
