File: mouse-joystick-pcb/mouse-joystick-pcb.kicad_sch (KiCad schematic)
At the start: 0 parts

Commit message: Update documentation for future v1.1
Other:
- company: Peter Polidoro -> Janelia Research Campus
Changed lines of the file:
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@@
 	(title_block
 		(title "mouse-joystick-pcb")
-		(date "2024-10-24")
-		(rev "1.0")
-		(company "Peter Polidoro")
+		(date "2026-01-15")
+		(rev "1.1")
+		(company "Janelia Research Campus")
+		(comment 1 "Peter Polidoro")
 	)
 	(wire
