File: mouse-joystick-pcb/power.kicad_sch (KiCad schematic)
At the start: 11 parts, among them Q301 MOSFET-N-CH-EN_100V_260mA, Q302 MOSFET-P-CH-EN_60V_50A, T301 TERM_BLK_HDR_2POS_90DEG_0.2IN, U301 TPSM365R6V5RDNR

Commit message: Make schematic changes
Connections:
- net VCC: no longer C303.1, U301.11 (MODE_SYNC), U301.8 (VCC)
- new net VDD: C303.1, U301.11 (MODE_SYNC), U301.8 (VCC)
Other:
- moved on the sheet: D301, Q301, Q302, R301, R302, T301

Commit message: Add components
Parts:
- removed C301: 3.3uF_50V, Janelia:C_1210_3225Metric, symbol Janelia:C_3.3uF_50V_1210
- removed C302: 0.1uF_100V, Janelia:C_0402_1005Metric, symbol Janelia:C_0.1uF_100V_0402
- removed C303, C304: 1uF_25V, Janelia:C_0402_1005Metric, symbol Janelia:C_1uF_25V_0402
- removed D301: D_50V_15A, Janelia:POWERDI5_DIO, symbol Janelia:D_50V_15A
- removed Q301: MOSFET-N-CH-EN_100V_260mA, Janelia:SOT-23, symbol Janelia:MOSFET-N-CH-EN_100V_260mA
- removed Q302: MOSFET-P-CH-EN_60V_50A, Janelia:TO-252-2, symbol Janelia:MOSFET-P-CH-EN_60V_50A
- removed R301: 1k, Janelia:R_0402_1005Metric, symbol Janelia:R_1k_0402
- removed R302: 3.6k, Janelia:R_0402_1005Metric, symbol Janelia:R_3.6k_0402
- removed T301: TERM_BLK_HDR_2POS_90DEG_0.2IN, Janelia:PHOENIX_1757242, symbol Janelia:TERM_BLK_HDR_2POS_90DEG_0.2IN
- removed U301: TPSM365R6V5RDNR, Janelia:RDN0011A-MFG, symbol Janelia:TPSM365R6V5RDNR
- added C14: 3.3uF_50V, Janelia:C_1210_3225Metric, symbol Janelia:C_3.3uF_50V_1210
- added C15: 0.1uF_100V, Janelia:C_0402_1005Metric, symbol Janelia:C_0.1uF_100V_0402
- added C16, C17: 1uF_25V, Janelia:C_0402_1005Metric, symbol Janelia:C_1uF_25V_0402
- added C18: 47uF_10V, Janelia:C_0805_2012Metric, symbol Janelia:C_47uF_10V_0805
- added D1: D_50V_15A, Janelia:POWERDI5_DIO, symbol Janelia:D_50V_15A
- added D2: LED_RED, Janelia:LED_0402-1005_KNB, symbol Janelia:LED_KNB_20mA_RED_1.95V_0402
- added R3: 2.32k, Janelia:R_0805_2012Metric, symbol Janelia:R_2.32k_1W_0805
- added U3: TPSM365R6V5RDNR, Janelia:RDN0011A-MFG, symbol Janelia:TPSM365R6V5RDNR
Connections:
- net +5V: now also C17.1, C18.1, U3.4 (VOUT), U3.9 (BIAS)
- net GND: now also C14.2, C15.2, C16.2, C17.2, C18.2, D2.1 (K), U3.10 (GND)
- net VAA: now also D1.2 (A)
- net VBB: now also C14.1, C15.1, D1.1 (K), R3.1, U3.2 (EN), U3.3 (VIN)
- net VDD: now also C16.1, U3.11 (MODE_SYNC), U3.8 (VCC)
- new net LED_RED+: D2.2 (A), R3.2

Commit message: Adjust schmatic
Parts:
- renumbered C14 to C301, C15 to C302, C16 to C303, C17 to C304, C18 to C305, D1 to D301, D2 to D302, R3 to R301, U3 to U301
Changed lines of the file:
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@@
   (symbol (lib_id "Janelia:C_3.3uF_50V_1210") (at 80.01 120.65 0) (unit 1)
     (in_bom yes) (on_board yes) (dnp no)
-    (property "Reference" "C14" (at 82.55 119.38 0)
+    (property "Reference" "C301" (at 82.55 119.38 0)
       (effects (font (size 1.016 1.016)) (justify left))
     )
@@
       (project "mouse-joystick-pcb"
         (path "/df2b2e89-e055-4140-95de-f1df723db034/c1dd8f61-494c-402f-8e59-08309c64fc3f"
-          (reference "C14") (unit 1)
+          (reference "C301") (unit 1)
         )
       )
@@
   (symbol (lib_id "power:PWR_FLAG") (at 130.81 45.72 0) (unit 1)
     (in_bom yes) (on_board yes) (dnp no)
-    (property "Reference" "#FLG01" (at 130.81 43.815 0)
+    (property "Reference" "#FLG0301" (at 130.81 43.815 0)
       (effects (font (size 1.27 1.27)) hide)
     )
@@
       (project "mouse-joystick-pcb"
         (path "/df2b2e89-e055-4140-95de-f1df723db034/c1dd8f61-494c-402f-8e59-08309c64fc3f"
-          (reference "#FLG01") (unit 1)
+          (reference "#FLG0301") (unit 1)
         )
       )
@@
   (symbol (lib_id "power:PWR_FLAG") (at 165.1 45.72 0) (unit 1)
     (in_bom yes) (on_board yes) (dnp no)
-    (property "Reference" "#FLG04" (at 165.1 43.815 0)
+    (property "Reference" "#FLG0304" (at 165.1 43.815 0)
       (effects (font (size 1.27 1.27)) hide)
     )
@@
       (project "mouse-joystick-pcb"
         (path "/df2b2e89-e055-4140-95de-f1df723db034/c1dd8f61-494c-402f-8e59-08309c64fc3f"
-          (reference "#FLG04") (unit 1)
+          (reference "#FLG0304") (unit 1)
         )
       )
@@
   (symbol (lib_id "Janelia:D_50V_15A") (at 165.1 67.31 180) (unit 1)
     (in_bom yes) (on_board yes) (dnp no) (fields_autoplaced)
-    (property "Reference" "D1" (at 165.1 60.96 0)
+    (property "Reference" "D301" (at 165.1 60.96 0)
       (effects (font (size 1.27 1.27)))
     )
@@
       (project "mouse-joystick-pcb"
         (path "/df2b2e89-e055-4140-95de-f1df723db034/c1dd8f61-494c-402f-8e59-08309c64fc3f"
-          (reference "D1") (unit 1)
+          (reference "D301") (unit 1)
         )
       )
@@
   (symbol (lib_id "Janelia:C_1uF_25V_0402") (at 109.22 120.65 0) (unit 1)
     (in_bom yes) (on_board yes) (dnp no)
-    (property "Reference" "C16" (at 111.76 119.38 0)
+    (property "Reference" "C303" (at 111.76 119.38 0)
       (effects (font (size 1.016 1.016)) (justify left))
     )
@@
       (project "mouse-joystick-pcb"
         (path "/df2b2e89-e055-4140-95de-f1df723db034/c1dd8f61-494c-402f-8e59-08309c64fc3f"
-          (reference "C16") (unit 1)
+          (reference "C303") (unit 1)
         )
       )
@@
   (symbol (lib_id "Janelia:LED_KNB_20mA_RED_1.95V_0402") (at 187.96 72.39 90) (unit 1)
     (in_bom yes) (on_board yes) (dnp no)
-    (property "Reference" "D2" (at 191.77 72.7075 90)
+    (property "Reference" "D302" (at 191.77 72.7075 90)
       (effects (font (size 1.27 1.27)) (justify right))
     )
@@
       (project "mouse-joystick-pcb"
         (path "/df2b2e89-e055-4140-95de-f1df723db034/c1dd8f61-494c-402f-8e59-08309c64fc3f"
-          (reference "D2") (unit 1)
+          (reference "D302") (unit 1)
         )
       )
@@
   (symbol (lib_id "power:PWR_FLAG") (at 153.67 45.72 0) (unit 1)
     (in_bom yes) (on_board yes) (dnp no)
-    (property "Reference" "#FLG03" (at 153.67 43.815 0)
+    (property "Reference" "#FLG0303" (at 153.67 43.815 0)
       (effects (font (size 1.27 1.27)) hide)
     )
@@
       (project "mouse-joystick-pcb"
         (path "/df2b2e89-e055-4140-95de-f1df723db034/c1dd8f61-494c-402f-8e59-08309c64fc3f"
-          (reference "#FLG03") (unit 1)
+          (reference "#FLG0303") (unit 1)
         )
       )
@@
   (symbol (lib_id "Janelia:C_47uF_10V_0805") (at 208.28 120.65 0) (unit 1)
     (in_bom yes) (on_board yes) (dnp no)
-    (property "Reference" "C18" (at 210.82 118.11 0)
+    (property "Reference" "C305" (at 210.82 118.11 0)
       (effects (font (size 1.016 1.016)) (justify left))
     )
@@
       (project "mouse-joystick-pcb"
         (path "/df2b2e89-e055-4140-95de-f1df723db034/c1dd8f61-494c-402f-8e59-08309c64fc3f"
-          (reference "C18") (unit 1)
+          (reference "C305") (unit 1)
         )
       )
@@
   (symbol (lib_id "Janelia:C_1uF_25V_0402") (at 195.58 120.65 0) (unit 1)
     (in_bom yes) (on_board yes) (dnp no)
-    (property "Reference" "C17" (at 198.12 118.11 0)
+    (property "Reference" "C304" (at 198.12 118.11 0)
       (effects (font (size 1.016 1.016)) (justify left))
     )
@@
       (project "mouse-joystick-pcb"
         (path "/df2b2e89-e055-4140-95de-f1df723db034/c1dd8f61-494c-402f-8e59-08309c64fc3f"
-          (reference "C17") (unit 1)
+          (reference "C304") (unit 1)
         )
       )
@@
   (symbol (lib_id "power:PWR_FLAG") (at 142.24 45.72 0) (unit 1)
     (in_bom yes) (on_board yes) (dnp no)
-    (property "Reference" "#FLG02" (at 142.24 43.815 0)
+    (property "Reference" "#FLG0302" (at 142.24 43.815 0)
       (effects (font (size 1.27 1.27)) hide)
     )
@@
       (project "mouse-joystick-pcb"
         (path "/df2b2e89-e055-4140-95de-f1df723db034/c1dd8f61-494c-402f-8e59-08309c64fc3f"
-          (reference "#FLG02") (unit 1)
+          (reference "#FLG0302") (unit 1)
         )
       )
@@
   (symbol (lib_id "Janelia:R_2.32k_1W_0805") (at 187.96 59.69 0) (unit 1)
     (in_bom yes) (on_board yes) (dnp no)
-    (property "Reference" "R3" (at 190.5 59.69 90)
+    (property "Reference" "R301" (at 190.5 59.69 90)
       (effects (font (size 1.016 1.016)))
     )
@@
       (project "mouse-joystick-pcb"
         (path "/df2b2e89-e055-4140-95de-f1df723db034/c1dd8f61-494c-402f-8e59-08309c64fc3f"
-          (reference "R3") (unit 1)
+          (reference "R301") (unit 1)
         )
       )
@@
   (symbol (lib_id "Janelia:TPSM365R6V5RDNR") (at 156.21 121.92 0) (unit 1)
     (in_bom yes) (on_board yes) (dnp no) (fields_autoplaced)
-    (property "Reference" "U3" (at 172.72 105.41 0) (do_not_autoplace)
+    (property "Reference" "U301" (at 172.72 105.41 0) (do_not_autoplace)
       (effects (font (size 1.524 1.524)))
     )
@@
       (project "mouse-joystick-pcb"
         (path "/df2b2e89-e055-4140-95de-f1df723db034/c1dd8f61-494c-402f-8e59-08309c64fc3f"
-          (reference "U3") (unit 1)
+          (reference "U301") (unit 1)
         )
       )
@@
   (symbol (lib_id "Janelia:C_0.1uF_100V_0402") (at 92.71 120.65 0) (unit 1)
     (in_bom yes) (on_board yes) (dnp no)
-    (property "Reference" "C15" (at 95.25 119.38 0)
+    (property "Reference" "C302" (at 95.25 119.38 0)
       (effects (font (size 1.016 1.016)) (justify left))
     )
@@
       (project "mouse-joystick-pcb"
         (path "/df2b2e89-e055-4140-95de-f1df723db034/c1dd8f61-494c-402f-8e59-08309c64fc3f"
-          (reference "C15") (unit 1)
-        )
-      )
+          (reference "C302") (unit 1)
+        )
+      )

Commit message: Start wiring schematics
Parts:
- added J301: 2.1, Janelia:Connector_BarrelJack_XKB_2.1, symbol Janelia:Barrel_Jack_Switch_SMD_RA_2.1_XKB
Connections:
- net GND: now also J301.2
- net VAA: now also J301.1
- no-connect marks 4 -> 5
Changed lines of the file:
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@@
   (no_connect (at 180.34 119.38))
   (no_connect (at 180.34 116.84))
+  (no_connect (at 130.81 68.58))
   (no_connect (at 132.08 129.54))
   (no_connect (at 180.34 111.76))
@@
     (stroke (width 0) (type default))
   )
-  (wire (pts (xy 132.08 68.58) (xy 134.62 68.58))
+  (wire (pts (xy 130.81 71.12) (xy 133.35 71.12))
     (stroke (width 0) (type default))
   )
@@
     (stroke (width 0) (type default))
   )
-  (wire (pts (xy 132.08 66.04) (xy 134.62 66.04))
+  (wire (pts (xy 130.81 66.04) (xy 133.35 66.04))
     (stroke (width 0) (type default))
   )
@@
     (stroke (width 0) (type default))
   )
-  (label "GND" (at 134.62 68.58 0) (fields_autoplaced)
+  (label "GND" (at 133.35 71.12 0) (fields_autoplaced)
     (effects (font (size 1.27 1.27)) (justify left bottom))
   )
@@
     (effects (font (size 1.27 1.27)) (justify right bottom))
   )
-  (label "VAA" (at 134.62 66.04 0) (fields_autoplaced)
+  (label "VAA" (at 133.35 66.04 0) (fields_autoplaced)
     (effects (font (size 1.27 1.27)) (justify left bottom))
   )
@@
         )
       )
+    )
+  )
+  (symbol (lib_id "Janelia:Barrel_Jack_Switch_SMD_RA_2.1_XKB") (at 123.19 68.58 0) (unit 1)
+    (in_bom yes) (on_board yes) (dnp no) (fields_autoplaced)
+    (property "Reference" "J301" (at 123.19 63.246 0) (do_not_autoplace)
+      (effects (font (size 1.27 1.27)))
+    )
+    (property "Value" "2.1" (at 123.19 73.66 0) (do_not_autoplace)
+      (effects (font (size 1.27 1.27)))
+    )
+    (property "Footprint" "Janelia:Connector_BarrelJack_XKB_2.1" (at 124.46 69.596 0)
+      (effects (font (size 1.27 1.27)) hide)
+    )
+    (property "Datasheet" "~" (at 124.46 69.596 0)
+      (effects (font (size 1.27 1.27)) hide)
+    )
+    (property "Synopsis" "DC Power Jack 2.5A 24V 2.1MM" (at 123.19 68.58 0)
+      (effects (font (size 1.27 1.27)) hide)
+    )
+    (property "Package" "SMD" (at 123.19 68.58 0)
+      (effects (font (size 1.27 1.27)) hide)
+    )
+    (property "Manufacturer" "XKB Connection" (at 123.19 68.58 0)
+      (effects (font (size 1.27 1.27)) hide)
+    )
+    (property "Manufacturer Part Number" "DC-005-2.5A-2.0-SMT" (at 123.19 68.58 0)
+      (effects (font (size 1.27 1.27)) hide)
+    )
+    (property "Vendor" "JLCPCB" (at 123.19 68.58 0)
+      (effects (font (size 1.27 1.27)) hide)
+    )
+    (property "Vendor Part Number" "C2880543" (at 123.19 68.58 0)
+      (effects (font (size 1.27 1.27)) hide)
+    )
+    (property "LCSC" "C2880543" (at 123.19 68.58 0)
+      (effects (font (size 1.27 1.27)) hide)
+    )
+    (pin "3")
+    (pin "2")
+    (pin "1")
+    (instances
+      (project "mouse-joystick-pcb"
+        (path "/df2b2e89-e055-4140-95de-f1df723db034/c1dd8f61-494c-402f-8e59-08309c64fc3f"
+          (reference "J301") (unit 1)
+        )
+      )
