File: mouse-joystick-pcb/microcontroller.kicad_sch (KiCad schematic)
At the start: 2 parts

Commit message: Add components
Parts:
- removed A401: PICO_W5500_EVB, Janelia:Pico-W5500-EVB_Header_Holes, symbol Janelia:PICO-W5500-EVB_HEADER_HOLES
- removed D401: D_SCHOTTKY_20V_1A, Janelia:DIOM3616X98N, symbol Janelia:D_SCHOTTKY_20V_1A
- added A1: PICO_W5500_EVB, Janelia:Pico-W5500-EVB_Header_Holes, symbol Janelia:PICO-W5500-EVB_HEADER_HOLES
- added D3: D_SCHOTTKY_20V_1A, Janelia:SOD-123FL, symbol Janelia:D_SCHOTTKY_20V_1A
- added R4, R6: 1.8k, Janelia:R_0402_1005Metric, symbol Janelia:R_1.8k_0402
Connections:
- net +3.3V: now also A1.36 (3V3(OUT)), R4.1, R6.1
- net +5V: now also D3.2 (A)
- net GND: now also A1.38 (GND)
- net VSYS: now also A1.39 (VSYS), D3.1 (K)
- new net AUDIO: A1.34 (ADC2/GP28)
- new net PRISM_CIPO: A1.16 (UART0-TX/I2C0-SDA/SPI1-RX/GP12)
- new net PRISM_COPI: A1.15 (I2C1-SCL/SPI1-TX/GP11)
- new net PRISM_SCK: A1.14 (I2C1-SDA/SPI1-SCK/GP10)
- new net SCL: A1.32 (I2C1-SCL/ADC1/GP27), R4.2
- new net SDA: A1.31 (I2C1-SDA/ADC0/GP26), R6.2
- new net ~{ADDRESS_INT}: A1.2 (UART0-RX/I2C0-SCL/SPI0-CS/GP1)
- new net ~{ADDRESS_RESET}: A1.1 (UART0-TX/I2C0-SDA/SPI0-RX/GP0)
- new net ~{PRISMS_RESET}: A1.20 (I2C1-SCL/SPI1-TX/GP15)
- new net ~{PRISM_CS_0}: A1.19 (I2C1-SDA/SPI1-SCK/GP14)
- new net ~{PRISM_CS_1}: A1.11 (UART1-TX/I2C0-SDA/SPI1-RX/GP8)
- new net ~{PRISM_CS_2}: A1.10 (I2C1-SCL/SPI0-TX/GP7)
- new net ~{PRISM_CS_3}: A1.9 (I2C1-SDA/SPI0-SCK/GP6)
- new net ~{PRISM_CS_4}: A1.7 (UART1-RX/I2C0-SCL/SPI0-CS/GP5)
- new net ~{PRISM_CS_5}: A1.6 (UART1-TX/I2C0-SDA/SPI0-RX/GP4)
- new net ~{PRISM_CS_6}: A1.5 (I2C1-SCL/SPI0-TX/GP3)
- no-connect marks 14 -> 15

Commit message: Adjust schmatic
Parts:
- removed A1: PICO_W5500_EVB, Janelia:Pico-W5500-EVB_Header_Holes, symbol Janelia:PICO-W5500-EVB_HEADER_HOLES
- added A401: TEENSY_4.1_HEADERS, Janelia:TEENSY_4.1_HEADERS, symbol Janelia:TEENSY_4.1_HEADERS
- renumbered D3 to D401, R4 to R401, R6 to R402
Connections:
- no-connect marks 15 -> 13

Commit message: Start wiring schematics
Parts:
- removed D401: D_SCHOTTKY_20V_1A, Janelia:SOD-123FL, symbol Janelia:D_SCHOTTKY_20V_1A
Connections:
- net +3.3V: now also A401.3V3 (3.3v_(250_mA_max))
- net GND: now also A401.GND
- no-connect marks 13 -> 0
Changed lines of the file:
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@@
     (company "Peter Polidoro")
   )
-  (no_connect (at 27.94 186.69))
-  (no_connect (at 27.94 161.29))
-  (no_connect (at 62.23 109.22))
-  (no_connect (at 62.23 121.92))
-  (no_connect (at 27.94 151.13))
-  (no_connect (at 62.23 134.62))
-  (no_connect (at 27.94 168.91))
-  (no_connect (at 27.94 173.99))
-  (no_connect (at 62.23 119.38))
-  (no_connect (at 27.94 156.21))
-  (no_connect (at 27.94 143.51))
-  (no_connect (at 27.94 171.45))
-  (no_connect (at 62.23 132.08))
-  (wire (pts (xy 128.27 60.96) (xy 125.73 60.96))
-    (stroke (width 0) (type default))
-  )
-  (wire (pts (xy 133.35 60.96) (xy 135.89 60.96))
-    (stroke (width 0) (type default))
-  )
-  (wire (pts (xy 27.94 166.37) (xy 30.48 166.37))
-    (stroke (width 0) (type default))
-  )
-  (wire (pts (xy 59.69 137.16) (xy 62.23 137.16))
-    (stroke (width 0) (type default))
-  )
-  (wire (pts (xy 59.69 104.14) (xy 62.23 104.14))
-    (stroke (width 0) (type default))
-  )
   (wire (pts (xy 50.8 52.07) (xy 53.34 52.07))
     (stroke (width 0) (type default))
@@
     (stroke (width 0) (type default))
   )
-  (wire (pts (xy 59.69 116.84) (xy 62.23 116.84))
-    (stroke (width 0) (type default))
-  )
   (wire (pts (xy 227.33 91.44) (xy 227.33 93.98))
     (stroke (width 0) (type default))
   )
-  (wire (pts (xy 27.94 153.67) (xy 30.48 153.67))
-    (stroke (width 0) (type default))
-  )
-  (wire (pts (xy 59.69 111.76) (xy 62.23 111.76))
+  (wire (pts (xy 162.56 82.55) (xy 165.1 82.55))
     (stroke (width 0) (type default))
   )
@@
     (stroke (width 0) (type default))
   )
-  (wire (pts (xy 59.69 124.46) (xy 62.23 124.46))
-    (stroke (width 0) (type default))
-  )
   (wire (pts (xy 50.8 49.53) (xy 53.34 49.53))
     (stroke (width 0) (type default))
   )
-  (wire (pts (xy 27.94 163.83) (xy 30.48 163.83))
-    (stroke (width 0) (type default))
-  )
-  (wire (pts (xy 59.69 101.6) (xy 62.23 101.6))
-    (stroke (width 0) (type default))
-  )
-  (wire (pts (xy 59.69 127) (xy 62.23 127))
-    (stroke (width 0) (type default))
-  )
-  (wire (pts (xy 50.8 46.99) (xy 53.34 46.99))
-    (stroke (width 0) (type default))
-  )
   (wire (pts (xy 50.8 57.15) (xy 53.34 57.15))
     (stroke (width 0) (type default))
   )
-  (wire (pts (xy 27.94 148.59) (xy 30.48 148.59))
-    (stroke (width 0) (type default))
-  )
-  (wire (pts (xy 59.69 139.7) (xy 62.23 139.7))
-    (stroke (width 0) (type default))
-  )
-  (wire (pts (xy 27.94 158.75) (xy 30.48 158.75))
-    (stroke (width 0) (type default))
-  )
   (wire (pts (xy 227.33 78.74) (xy 227.33 76.2))
     (stroke (width 0) (type default))
   )
-  (wire (pts (xy 59.69 129.54) (xy 62.23 129.54))
-    (stroke (width 0) (type default))
-  )
   (wire (pts (xy 218.44 91.44) (xy 218.44 93.98))
     (stroke (width 0) (type default))
   )
-  (wire (pts (xy 27.94 146.05) (xy 30.48 146.05))
-    (stroke (width 0) (type default))
-  )
   (wire (pts (xy 218.44 78.74) (xy 218.44 76.2))
     (stroke (width 0) (type default))
   )
-  (wire (pts (xy 59.69 114.3) (xy 62.23 114.3))
-    (stroke (width 0) (type default))
-  )
-  (wire (pts (xy 59.69 106.68) (xy 62.23 106.68))
-    (stroke (width 0) (type default))
-  )
-  (label "+3.3V" (at 30.48 153.67 0) (fields_autoplaced)
+  (wire (pts (xy 99.06 77.47) (xy 96.52 77.47))
+    (stroke (width 0) (type default))
+  )
+  (label "+3.3V" (at 165.1 82.55 0) (fields_autoplaced)
     (effects (font (size 1.27 1.27)) (justify left bottom))
   )
@@
     (effects (font (size 1.27 1.27)) (justify right bottom))
   )
-  (label "SDA" (at 30.48 166.37 0) (fields_autoplaced)
-    (effects (font (size 1.27 1.27)) (justify left bottom))
-  )
-  (label "SCL" (at 30.48 163.83 0) (fields_autoplaced)
-    (effects (font (size 1.27 1.27)) (justify left bottom))
-  )
   (label "GND" (at 53.34 52.07 0) (fields_autoplaced)
     (effects (font (size 1.27 1.27)) (justify left bottom))
   )
-  (label "GND" (at 30.48 148.59 0) (fields_autoplaced)
-    (effects (font (size 1.27 1.27)) (justify left bottom))
-  )
   (label "SCL" (at 218.44 93.98 270) (fields_autoplaced)
     (effects (font (size 1.27 1.27)) (justify right bottom))
   )
-  (label "VSYS" (at 135.89 60.96 0) (fields_autoplaced)
-    (effects (font (size 1.27 1.27)) (justify left bottom))
-  )
-  (label "VSYS" (at 30.48 146.05 0) (fields_autoplaced)
-    (effects (font (size 1.27 1.27)) (justify left bottom))
+  (label "GND" (at 96.52 77.47 180) (fields_autoplaced)
+    (effects (font (size 1.27 1.27)) (justify right bottom))
   )
   (label "VSYS" (at 187.96 52.07 270) (fields_autoplaced)
     (effects (font (size 1.27 1.27)) (justify right bottom))
   )
-  (label "+5V" (at 53.34 46.99 0) (fields_autoplaced)
-    (effects (font (size 1.27 1.27)) (justify left bottom))
-  )
   (label "SCL" (at 53.34 54.61 0) (fields_autoplaced)
     (effects (font (size 1.27 1.27)) (justify left bottom))
@@
     (effects (font (size 1.27 1.27)) (justify left bottom))
   )
-  (label "+5V" (at 125.73 60.96 180) (fields_autoplaced)
-    (effects (font (size 1.27 1.27)) (justify right bottom))
-  )
   (label "+3.3V" (at 53.34 49.53 0) (fields_autoplaced)
     (effects (font (size 1.27 1.27)) (justify left bottom))
@@
   (label "SDA" (at 53.34 57.15 0) (fields_autoplaced)
     (effects (font (size 1.27 1.27)) (justify left bottom))
-  )
-  (hierarchical_label "~{PRISM_CS_1}" (shape output) (at 59.69 116.84 180) (fields_autoplaced)
-    (effects (font (size 1.27 1.27)) (justify right))
-  )
-  (hierarchical_label "+5V" (shape passive) (at 50.8 46.99 180) (fields_autoplaced)
-    (effects (font (size 1.27 1.27)) (justify right))
-  )
-  (hierarchical_label "~{PRISM_CS_0}" (shape output) (at 59.69 137.16 180) (fields_autoplaced)
-    (effects (font (size 1.27 1.27)) (justify right))
-  )
-  (hierarchical_label "AUDIO" (shape output) (at 30.48 158.75 0) (fields_autoplaced)
-    (effects (font (size 1.27 1.27)) (justify left))
-  )
-  (hierarchical_label "PRISM_COPI" (shape output) (at 59.69 127 180) (fields_autoplaced)
-    (effects (font (size 1.27 1.27)) (justify right))
-  )
-  (hierarchical_label "~{PRISM_CS_6}" (shape output) (at 59.69 101.6 180) (fields_autoplaced)
-    (effects (font (size 1.27 1.27)) (justify right))
-  )
-  (hierarchical_label "PRISM_CIPO" (shape input) (at 59.69 129.54 180) (fields_autoplaced)
-    (effects (font (size 1.27 1.27)) (justify right))
-  )
-  (hierarchical_label "~{PRISM_CS_5}" (shape output) (at 59.69 104.14 180) (fields_autoplaced)
-    (effects (font (size 1.27 1.27)) (justify right))
   )
   (hierarchical_label "GND" (shape passive) (at 50.8 52.07 180) (fields_autoplaced)
     (effects (font (size 1.27 1.27)) (justify right))
   )
-  (hierarchical_label "~{PRISM_CS_2}" (shape output) (at 59.69 114.3 180) (fields_autoplaced)
-    (effects (font (size 1.27 1.27)) (justify right))
-  )
   (hierarchical_label "+3.3V" (shape passive) (at 50.8 49.53 180) (fields_autoplaced)
     (effects (font (size 1.27 1.27)) (justify right))
@@
   )
   (hierarchical_label "SCL" (shape output) (at 50.8 54.61 180) (fields_autoplaced)
-    (effects (font (size 1.27 1.27)) (justify right))
-  )
-  (hierarchical_label "PRISM_SCK" (shape output) (at 59.69 124.46 180) (fields_autoplaced)
-    (effects (font (size 1.27 1.27)) (justify right))
-  )
-  (hierarchical_label "~{PRISM_CS_3}" (shape output) (at 59.69 111.76 180) (fields_autoplaced)
-    (effects (font (size 1.27 1.27)) (justify right))
-  )
-  (hierarchical_label "~{PRISMS_RESET}" (shape output) (at 59.69 139.7 180) (fields_autoplaced)
-    (effects (font (size 1.27 1.27)) (justify right))
-  )
-  (hierarchical_label "~{PRISM_CS_4}" (shape output) (at 59.69 106.68 180) (fields_autoplaced)
     (effects (font (size 1.27 1.27)) (justify right))
   )
@@
         )
       )
-    )
-  )
-  (symbol (lib_id "Janelia:D_SCHOTTKY_20V_1A") (at 130.81 60.96 180) (unit 1)
-    (in_bom yes) (on_board yes) (dnp no) (fields_autoplaced)
-    (property "Reference" "D401" (at 130.937 57.15 0)
-      (effects (font (size 1.27 1.27)))
-    )
-    (property "Value" "D_SCHOTTKY_20V_1A" (at 137.922 58.928 0)
-      (effects (font (size 1.27 1.27)) (justify left) hide)
-    )
-    (property "Footprint" "Janelia:SOD-123FL" (at 134.62 60.452 0)
-      (effects (font (size 1.524 1.524)) hide)
-    )
-    (property "Datasheet" "" (at 132.08 62.992 0)
-      (effects (font (size 1.524 1.524)) hide)
-    )
-    (property "Vendor" "Digi-Key" (at 129.54 65.532 0)
-      (effects (font (size 1.524 1.524)) hide)
-    )
-    (property "Vendor Part Number" "MBR120VLSFT1GOSCT-ND" (at 127 68.072 0)
-      (effects (font (size 1.524 1.524)) hide)
-    )
-    (property "Synopsis" "DIODE SCHOTTKY 20V 1A" (at 124.46 70.612 0)
-      (effects (font (size 1.524 1.524)) hide)
-    )
-    (property "Manufacturer" "onsemi" (at 130.81 60.96 0)
-      (effects (font (size 1.27 1.27)) hide)
-    )
-    (property "Manufacturer Part Number" "MBR120VLSFT1G" (at 130.81 60.96 0)
-      (effects (font (size 1.27 1.27)) hide)
-    )
-    (property "Package" "SOD-123FL" (at 130.81 60.96 0)
-      (effects (font (size 1.27 1.27)) hide)
-    )
-    (property "Sim.Enable" "0" (at 130.81 60.96 0)
-      (effects (font (size 1.27 1.27)) hide)
-    )
-    (property "LCSC" "C223608" (at 130.81 60.96 0)
-      (effects (font (size 1.27 1.27)) hide)
-    )
-    (pin "1")
-    (pin "2")
-    (instances
-      (project "mouse-joystick-pcb"
-        (path "/df2b2e89-e055-4140-95de-f1df723db034/90ad6836-1738-4b32-a341-0a0b169f4662"
-          (reference "D401") (unit 1)
-        )
-      )

Commit message: Finish v1.0 schematic
Parts:
- removed A401: TEENSY_4.1_HEADERS, Janelia:TEENSY_4.1_HEADERS, symbol Janelia:TEENSY_4.1_HEADERS
- removed R401, R402: 1.8k, Janelia:R_0402_1005Metric, symbol Janelia:R_1.8k_0402
- added A401: TEENSY_4.0_HEADERS, Janelia:TEENSY_4.0_HEADERS, symbol Janelia:TEENSY_4.0_HEADERS
Connections:
- net +3.3V: now also A401.3V3 (3.3v_(250_mA_max))
- net GND: now also A401.GND
- new net AUDIO: A401.23 (D23/A9/CRX1/MCLK1/PWM)
- new net BRAKE_PWM: A401.22 (D22/A8/CTX1/PWM)
- new net CIPO: A401.12 (D12/CIPO/MQSL/PWM)
- new net COPI: A401.11 (D11/COPI/PWM)
- new net MOTOR_DIAG0_0: A401.15 (D15/A1/RX3/SIN/PWM)
- new net MOTOR_DIAG0_1: A401.19 (D19/A5/SCL0/PWM)
- new net SCK: A401.13 (D13/LED/SCK/PWM)
- new net ~{MOTOR_CS_0}: A401.14 (D14/A0/TX3/SOUT/PWM)
- new net ~{MOTOR_CS_1}: A401.18 (D18/A4/SDA0/PWM)
- no-connect marks 0 -> 16

Commit message: Initial footprint layout
Connections:
- net AUDIO: now also A401.9 (D9/OUT1C/PWM); no longer A401.23 (D23/A9/CRX1/MCLK1/PWM)
- net BRAKE_PWM: now also A401.10 (D10/CS/MQSR/PWM); no longer A401.22 (D22/A8/CTX1/PWM)
Changed lines of the file:
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@@
   (title_block
     (title "mouse-joystick-pcb")
-    (date "2024-10-08")
+    (date "2024-10-09")
     (rev "1.0")
     (company "Peter Polidoro")
@@
   (no_connect (at 99.06 87.63))
   (no_connect (at 99.06 90.17))
-  (no_connect (at 99.06 102.87))
-  (no_connect (at 99.06 105.41))
+  (no_connect (at 162.56 85.09))
+  (no_connect (at 162.56 87.63))
   (wire (pts (xy 162.56 110.49) (xy 165.1 110.49))
     (stroke (width 0) (type default))
@@
     (stroke (width 0) (type default))
   )
-  (wire (pts (xy 162.56 87.63) (xy 165.1 87.63))
-    (stroke (width 0) (type default))
-  )
-  (wire (pts (xy 162.56 85.09) (xy 165.1 85.09))
+  (wire (pts (xy 99.06 102.87) (xy 96.52 102.87))
     (stroke (width 0) (type default))
   )
@@
     (stroke (width 0) (type default))
   )
+  (wire (pts (xy 96.52 105.41) (xy 99.06 105.41))
+    (stroke (width 0) (type default))
+  )
   (wire (pts (xy 99.06 77.47) (xy 96.52 77.47))
     (stroke (width 0) (type default))
@@
     (effects (font (size 1.27 1.27)) (justify left))
   )
-  (hierarchical_label "BRAKE_PWM" (shape output) (at 165.1 87.63 0) (fields_autoplaced)
-    (effects (font (size 1.27 1.27)) (justify left))
+  (hierarchical_label "BRAKE_PWM" (shape output) (at 96.52 105.41 180) (fields_autoplaced)
+    (effects (font (size 1.27 1.27)) (justify right))
   )
   (hierarchical_label "MOTOR_DIAG0_1" (shape input) (at 165.1 95.25 0) (fields_autoplaced)
@@
     (effects (font (size 1.27 1.27)) (justify left))
   )
-  (hierarchical_label "AUDIO" (shape output) (at 165.1 85.09 0) (fields_autoplaced)
-    (effects (font (size 1.27 1.27)) (justify left))
+  (hierarchical_label "AUDIO" (shape output) (at 96.52 102.87 180) (fields_autoplaced)
+    (effects (font (size 1.27 1.27)) (justify right))
   )
   (hierarchical_label "MOTOR_DIAG0_0" (shape input) (at 165.1 105.41 0) (fields_autoplaced)
