File: mouse-joystick-pcb/brake.kicad_sch (KiCad schematic)
At the start: 0 parts

Commit message: Adjust schmatic
Parts:
- added U801: 40V_200mA, Janelia:SC-74-6_1.55x2.9mm_P0.95mm, symbol Janelia:LED_DRIVER_LINEAR_BCR421U
Connections:
- new net: U801.2 (IOUT), U801.3 (IOUT), U801.5 (IOUT)
Changed lines of the file:
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@@
 (kicad_sch (version 20230121) (generator eeschema)
   (paper "A4")
+  (symbol (lib_id "Janelia:LED_DRIVER_LINEAR_BCR421U") (at 138.43 88.9 0) (unit 1)
+    (in_bom yes) (on_board yes) (dnp no) (fields_autoplaced)
+    (property "Reference" "U801" (at 138.43 78.74 0) (do_not_autoplace)
+      (effects (font (size 1.27 1.27)))
+    )
+    (property "Value" "40V_200mA" (at 158.75 63.5 0)
+      (effects (font (size 1.27 1.27)) (justify left) hide)
+    )
+    (property "Footprint" "Janelia:SC-74-6_1.55x2.9mm_P0.95mm" (at 138.43 68.58 0)
+      (effects (font (size 1.27 1.27)) hide)
+    )
+    (property "Datasheet" "~" (at 138.43 63.5 0)
+      (effects (font (size 1.27 1.27)) hide)
+    )
+    (property "Synopsis" "IC LED DRVR LIN PWM 200MA" (at 138.43 66.04 0)
+      (effects (font (size 1.27 1.27)) hide)
+    )
+    (property "Package" "SC-74-6" (at 138.43 73.66 0)
+      (effects (font (size 1.27 1.27)) hide)
+    )
+    (property "Manufacturer" "Infineon Technologies" (at 138.43 55.88 0)
+      (effects (font (size 1.27 1.27)) hide)
+    )
+    (property "Manufacturer Part Number" "BCR421UE6327" (at 138.43 60.96 0)
+      (effects (font (size 1.27 1.27)) hide)
+    )
+    (property "Vendor" "Digi-Key" (at 138.43 58.42 0)
+      (effects (font (size 1.27 1.27)) hide)
+    )
+    (property "Vendor Part Number" "BCR421UE6327HTSA1CT-ND" (at 138.43 71.12 0)
+      (effects (font (size 1.27 1.27)) hide)
+    )
+    (property "Sim.Enable" "0" (at 138.43 88.9 0)
+      (effects (font (size 1.27 1.27)) hide)
+    )
+    (property "LCSC" "C112923" (at 138.43 88.9 0)
+      (effects (font (size 1.27 1.27)) hide)
+    )
+    (pin "5")
+    (pin "6")
+    (pin "2")
+    (pin "1")
+    (pin "3")
+    (pin "4")
+    (instances
+      (project "mouse-joystick-pcb"
+        (path "/df2b2e89-e055-4140-95de-f1df723db034/cc53e4cb-28ca-4497-a17f-97087cae7de9"
+          (reference "U801") (unit 1)
+        )
+      )
+    )
+  )
 )

Commit message: Update date
Parts:
- added R801: 30, Janelia:R_0402_1005Metric, symbol Janelia:R_30_0402
Other:
- note added: "30Ohm ~ 40mA ~ 2.6newton-cm"
- company: (none) -> Peter Polidoro
- title: (none) -> mouse-joystick-pcb
Changed lines of the file:
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@@
 (kicad_sch (version 20230121) (generator eeschema)
   (paper "A4")
+  (title_block
+    (title "mouse-joystick-pcb")
+    (date "2024-10-07")
+    (rev "1.0")
+    (company "Peter Polidoro")
+  )
+  (text "30Ohm ~ 40mA ~ 2.6newton-cm" (at 163.83 101.6 0)
+    (effects (font (size 1.27 1.27)) (justify left bottom))
+  )
   (symbol (lib_id "Janelia:LED_DRIVER_LINEAR_BCR421U") (at 138.43 88.9 0) (unit 1)
     (in_bom yes) (on_board yes) (dnp no) (fields_autoplaced)
@@
         )
       )
+    )
+  )
+  (symbol (lib_id "Janelia:R_30_0402") (at 157.48 100.33 0) (unit 1)
+    (in_bom yes) (on_board yes) (dnp no) (fields_autoplaced)
+    (property "Reference" "R801" (at 158.75 100.33 0) (do_not_autoplace)
+      (effects (font (size 1.016 1.016)) (justify left))
+    )
+    (property "Value" "30" (at 157.48 100.33 90) (do_not_autoplace)
+      (effects (font (size 0.762 0.762)))
+    )
+    (property "Footprint" "Janelia:R_0402_1005Metric" (at 155.702 100.33 90)
+      (effects (font (size 0.762 0.762)) hide)
+    )
+    (property "Datasheet" "" (at 159.512 100.33 90)
+      (effects (font (size 0.762 0.762)) hide)
+    )
+    (property "Vendor" "JLCPCB" (at 162.052 97.79 90)
+      (effects (font (size 1.524 1.524)) hide)
+    )
+    (property "Vendor Part Number" "C3036820" (at 164.592 95.25 90)
+      (effects (font (size 1.524 1.524)) hide)
+    )
+    (property "Synopsis" "RES 30 OHM 1% 62.5mW" (at 167.132 92.71 90)
+      (effects (font (size 1.524 1.524)) hide)
+    )
+    (property "Manufacturer" "LIZ Elec" (at 157.48 84.455 0)
+      (effects (font (size 1.27 1.27)) hide)
+    )
+    (property "Manufacturer Part Number" "CR0402FF30R0G" (at 157.48 81.915 0)
+      (effects (font (size 1.27 1.27)) hide)
+    )
+    (property "Package" "0402" (at 157.48 80.01 0)
+      (effects (font (size 1.27 1.27)) hide)
+    )
+    (property "LCSC" "C3036820" (at 157.48 78.105 0)
+      (effects (font (size 1.27 1.27)) hide)
+    )
+    (pin "1")
+    (pin "2")
+    (instances
+      (project "mouse-joystick-pcb"
+        (path "/df2b2e89-e055-4140-95de-f1df723db034/cc53e4cb-28ca-4497-a17f-97087cae7de9"
+          (reference "R801") (unit 1)
+        )
+      )

Commit message: Start wiring schematics
Parts:
- added J801: Conn_01x02_P3.5mm_TBH_Horizontal_Screw, Janelia:PhoenixContact_MC_1,5_2-G-3.5_1x02_P3.50mm_Horizontal_Screw, symbol Janelia:Conn_01x02_P3.5mm_TBH_Horizontal_Screw
Connections:
- net IOUT: now reaches U801.2 (IOUT), U801.3 (IOUT), U801.5 (IOUT)
- net IOUT: now also J801.1 (Pin_1)
- net GND: now reaches U801.4 (GND)
- net GND: now also R801.2
- net at U801.6 (REXT): now also R801.1
- new net REFL: J801.2 (Pin_2)
Other:
- moved on the sheet: R801
Changed lines of the file:
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@@
     (company "Peter Polidoro")
   )
-  (text "30Ohm ~ 40mA ~ 2.6newton-cm" (at 163.83 101.6 0)
+  (wire (pts (xy 151.13 92.71) (xy 151.13 95.25))
+    (stroke (width 0) (type default))
+  )
+  (wire (pts (xy 148.59 82.55) (xy 151.13 82.55))
+    (stroke (width 0) (type default))
+  )
+  (wire (pts (xy 201.93 88.9) (xy 199.39 88.9))
+    (stroke (width 0) (type default))
+  )
+  (wire (pts (xy 138.43 102.87) (xy 138.43 105.41))
+    (stroke (width 0) (type default))
+  )
+  (wire (pts (xy 151.13 107.95) (xy 151.13 110.49))
+    (stroke (width 0) (type default))
+  )
+  (wire (pts (xy 201.93 86.36) (xy 199.39 86.36))
+    (stroke (width 0) (type default))
+  )
+  (wire (pts (xy 148.59 92.71) (xy 151.13 92.71))
+    (stroke (width 0) (type default))
+  )
+  (text "30Ohm ~ 40mA ~ 2.6newton-cm" (at 157.48 102.87 0)
     (effects (font (size 1.27 1.27)) (justify left bottom))
+  )
+  (label "IOUT" (at 199.39 88.9 180) (fields_autoplaced)
+    (effects (font (size 1.27 1.27)) (justify right bottom))
+  )
+  (label "GND" (at 138.43 105.41 270) (fields_autoplaced)
+    (effects (font (size 1.27 1.27)) (justify right bottom))
+  )
+  (label "IOUT" (at 151.13 82.55 0) (fields_autoplaced)
+    (effects (font (size 1.27 1.27)) (justify left bottom))
+  )
+  (label "REFL" (at 199.39 86.36 180) (fields_autoplaced)
+    (effects (font (size 1.27 1.27)) (justify right bottom))
+  )
+  (label "GND" (at 151.13 110.49 270) (fields_autoplaced)
+    (effects (font (size 1.27 1.27)) (justify right bottom))
   )
   (symbol (lib_id "Janelia:LED_DRIVER_LINEAR_BCR421U") (at 138.43 88.9 0) (unit 1)
@@
     )
   )
-  (symbol (lib_id "Janelia:R_30_0402") (at 157.48 100.33 0) (unit 1)
+  (symbol (lib_id "Janelia:Conn_01x02_P3.5mm_TBH_Horizontal_Screw") (at 207.01 88.9 180) (unit 1)
     (in_bom yes) (on_board yes) (dnp no) (fields_autoplaced)
-    (property "Reference" "R801" (at 158.75 100.33 0) (do_not_autoplace)
+    (property "Reference" "J801" (at 208.28 87.63 0)
+      (effects (font (size 1.27 1.27)) (justify right))
+    )
+    (property "Value" "Conn_01x02_P3.5mm_TBH_Horizontal_Screw" (at 207.01 76.2 0)
+      (effects (font (size 1.27 1.27)) hide)
+    )
+    (property "Footprint" "Janelia:PhoenixContact_MC_1,5_2-G-3.5_1x02_P3.50mm_Horizontal_Screw" (at 207.01 124.46 0)
+      (effects (font (size 1.27 1.27)) hide)
+    )
+    (property "Datasheet" "" (at 207.01 110.49 0)
+      (effects (font (size 1.27 1.27)) hide)
+    )
+    (property "Manufacturer" "Phoenix Contact" (at 207.01 121.92 0)
+      (effects (font (size 1.27 1.27)) hide)
+    )
+    (property "Manufacturer Part Number" "1844210" (at 207.01 116.84 0)
+      (effects (font (size 1.27 1.27)) hide)
+    )
+    (property "Synopsis" "TERM BLOCK HDR 2POS 90DEG 3.5MM" (at 207.01 114.3 0)
+      (effects (font (size 1.27 1.27)) hide)
+    )
+    (property "Vendor" "Digi-Key" (at 207.01 119.38 0)
+      (effects (font (size 1.27 1.27)) hide)
+    )
+    (property "Vendor Part Number" "277-2416-ND" (at 207.01 111.76 0)
+      (effects (font (size 1.27 1.27)) hide)
+    )
+    (property "Sim.Enable" "0" (at 207.01 88.9 0)
+      (effects (font (size 1.27 1.27)) hide)
+    )
+    (property "Package" "Plugin P=3.5mm" (at 207.01 88.9 0)
+      (effects (font (size 1.27 1.27)) hide)
+    )
+    (property "LCSC" "C3584780" (at 207.01 88.9 0)
+      (effects (font (size 1.27 1.27)) hide)
+    )
+    (pin "2")
+    (pin "1")
+    (instances
+      (project "mouse-joystick-pcb"
+        (path "/df2b2e89-e055-4140-95de-f1df723db034/cc53e4cb-28ca-4497-a17f-97087cae7de9"
+          (reference "J801") (unit 1)
+        )
+      )
+    )
+  )
+  (symbol (lib_id "Janelia:R_30_0402") (at 151.13 101.6 0) (unit 1)
+    (in_bom yes) (on_board yes) (dnp no) (fields_autoplaced)
+    (property "Reference" "R801" (at 152.4 101.6 0) (do_not_autoplace)
       (effects (font (size 1.016 1.016)) (justify left))
     )
-    (property "Value" "30" (at 157.48 100.33 90) (do_not_autoplace)
+    (property "Value" "30" (at 151.13 101.6 90) (do_not_autoplace)
       (effects (font (size 0.762 0.762)))
     )
-    (property "Footprint" "Janelia:R_0402_1005Metric" (at 155.702 100.33 90)
+    (property "Footprint" "Janelia:R_0402_1005Metric" (at 149.352 101.6 90)
       (effects (font (size 0.762 0.762)) hide)
     )
-    (property "Datasheet" "" (at 159.512 100.33 90)
+    (property "Datasheet" "" (at 153.162 101.6 90)
       (effects (font (size 0.762 0.762)) hide)
     )
-    (property "Vendor" "JLCPCB" (at 162.052 97.79 90)
+    (property "Vendor" "JLCPCB" (at 155.702 99.06 90)
       (effects (font (size 1.524 1.524)) hide)
     )
-    (property "Vendor Part Number" "C3036820" (at 164.592 95.25 90)
+    (property "Vendor Part Number" "C3036820" (at 158.242 96.52 90)
       (effects (font (size 1.524 1.524)) hide)
     )
-    (property "Synopsis" "RES 30 OHM 1% 62.5mW" (at 167.132 92.71 90)
+    (property "Synopsis" "RES 30 OHM 1% 62.5mW" (at 160.782 93.98 90)
       (effects (font (size 1.524 1.524)) hide)
     )
-    (property "Manufacturer" "LIZ Elec" (at 157.48 84.455 0)
+    (property "Manufacturer" "LIZ Elec" (at 151.13 85.725 0)
       (effects (font (size 1.27 1.27)) hide)
     )
-    (property "Manufacturer Part Number" "CR0402FF30R0G" (at 157.48 81.915 0)
+    (property "Manufacturer Part Number" "CR0402FF30R0G" (at 151.13 83.185 0)
       (effects (font (size 1.27 1.27)) hide)
     )
-    (property "Package" "0402" (at 157.48 80.01 0)
+    (property "Package" "0402" (at 151.13 81.28 0)
       (effects (font (size 1.27 1.27)) hide)
     )
-    (property "LCSC" "C3036820" (at 157.48 78.105 0)
+    (property "LCSC" "C3036820" (at 151.13 79.375 0)
       (effects (font (size 1.27 1.27)) hide)
     )

Commit message: Finish v1.0 schematic
Parts:
- added C801: 100uF_50V, Janelia:CAP_EEEHAH101UAP, symbol Janelia:CP_100uF_50V_8x10.2mm
Connections:
- net GND: now also C801.2
- net BRAKE_PWM: now reaches U801.1 (VEN)
- net REFL renamed VS
- net VS: now also C801.1
Other:
- note added: "30 Ohm ~ 40 mA ~ 2.6 newton-cm"
- note removed: "30Ohm ~ 40mA ~ 2.6newton-cm"
Changed lines of the file:
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@@
   (title_block
     (title "mouse-joystick-pcb")
-    (date "2024-10-07")
+    (date "2024-10-08")
     (rev "1.0")
     (company "Peter Polidoro")
   )
+  (wire (pts (xy 182.88 68.58) (xy 182.88 66.04))
+    (stroke (width 0) (type default))
+  )
   (wire (pts (xy 151.13 92.71) (xy 151.13 95.25))
+    (stroke (width 0) (type default))
+  )
+  (wire (pts (xy 182.88 73.66) (xy 182.88 76.2))
     (stroke (width 0) (type default))
   )
@@
     (stroke (width 0) (type default))
   )
+  (wire (pts (xy 88.9 49.53) (xy 91.44 49.53))
+    (stroke (width 0) (type default))
+  )
   (wire (pts (xy 201.93 86.36) (xy 199.39 86.36))
+    (stroke (width 0) (type default))
+  )
+  (wire (pts (xy 128.27 82.55) (xy 125.73 82.55))
+    (stroke (width 0) (type default))
+  )
+  (wire (pts (xy 88.9 46.99) (xy 91.44 46.99))
     (stroke (width 0) (type default))
   )
@@
     (stroke (width 0) (type default))
   )
-  (text "30Ohm ~ 40mA ~ 2.6newton-cm" (at 157.48 102.87 0)
+  (wire (pts (xy 88.9 52.07) (xy 91.44 52.07))
+    (stroke (width 0) (type default))
+  )
+  (text "30 Ohm ~ 40 mA ~ 2.6 newton-cm" (at 157.48 102.87 0)
+    (effects (font (size 1.27 1.27)) (justify left bottom))
+  )
+  (label "VS" (at 199.39 86.36 180) (fields_autoplaced)
+    (effects (font (size 1.27 1.27)) (justify right bottom))
+  )
+  (label "VS" (at 182.88 66.04 90) (fields_autoplaced)
     (effects (font (size 1.27 1.27)) (justify left bottom))
   )
@@
     (effects (font (size 1.27 1.27)) (justify left bottom))
   )
-  (label "REFL" (at 199.39 86.36 180) (fields_autoplaced)
+  (label "BRAKE_PWM" (at 125.73 82.55 180) (fields_autoplaced)
+    (effects (font (size 1.27 1.27)) (justify right bottom))
+  )
+  (label "GND" (at 182.88 76.2 270) (fields_autoplaced)
     (effects (font (size 1.27 1.27)) (justify right bottom))
   )
@@
     (effects (font (size 1.27 1.27)) (justify right bottom))
   )
+  (label "VS" (at 91.44 46.99 0) (fields_autoplaced)
+    (effects (font (size 1.27 1.27)) (justify left bottom))
+  )
+  (label "BRAKE_PWM" (at 91.44 52.07 0) (fields_autoplaced)
+    (effects (font (size 1.27 1.27)) (justify left bottom))
+  )
+  (label "GND" (at 91.44 49.53 0) (fields_autoplaced)
+    (effects (font (size 1.27 1.27)) (justify left bottom))
+  )
+  (hierarchical_label "GND" (shape passive) (at 88.9 49.53 180) (fields_autoplaced)
+    (effects (font (size 1.27 1.27)) (justify right))
+  )
+  (hierarchical_label "BRAKE_PWM" (shape input) (at 88.9 52.07 180) (fields_autoplaced)
+    (effects (font (size 1.27 1.27)) (justify right))
+  )
+  (hierarchical_label "VS" (shape passive) (at 88.9 46.99 180) (fields_autoplaced)
+    (effects (font (size 1.27 1.27)) (justify right))
+  )
+  (symbol (lib_id "Janelia:CP_100uF_50V_8x10.2mm") (at 182.88 71.12 0) (unit 1)
+    (in_bom yes) (on_board yes) (dnp no) (fields_autoplaced)
+    (property "Reference" "C801" (at 185.42 69.9389 0)
+      (effects (font (size 1.016 1.016)) (justify left))
+    )
+    (property "Value" "100uF_50V" (at 185.42 71.8438 0)
+      (effects (font (size 0.762 0.762)) (justify left))
+    )
+    (property "Footprint" "Janelia:CAP_EEEHAH101UAP" (at 180.594 71.882 0)
+      (effects (font (size 1.524 1.524)) hide)
+    )
+    (property "Datasheet" "" (at 183.134 69.342 0)
+      (effects (font (size 1.524 1.524)) hide)
+    )
+    (property "Vendor" "Digi-Key" (at 185.674 66.802 0)
+      (effects (font (size 1.524 1.524)) hide)
+    )
+    (property "Vendor Part Number" "PCE4713CT-ND" (at 188.214 64.262 0)
+      (effects (font (size 1.524 1.524)) hide)
+    )
+    (property "Synopsis" "CAP ALUM 100UF 20% 50V SMD" (at 190.754 61.722 0)
+      (effects (font (size 1.524 1.524)) hide)
+    )
+    (property "Manufacturer" "Panasonic Electronic Components" (at 182.88 71.12 0)
+      (effects (font (size 1.27 1.27)) hide)
+    )
+    (property "Manufacturer Part Number" "EEEHAH101UAP" (at 182.88 71.12 0)
+      (effects (font (size 1.27 1.27)) hide)
+    )
+    (property "LCSC" "C336425" (at 182.88 71.12 0)
+      (effects (font (size 1.27 1.27)) hide)
+    )
+    (property "Package" "SMD D8xL10.2mm" (at 182.88 71.12 0)
+      (effects (font (size 1.27 1.27)) hide)
+    )
+    (pin "2")
+    (pin "1")
+    (instances
+      (project "mouse-joystick-pcb"
+        (path "/df2b2e89-e055-4140-95de-f1df723db034/cc53e4cb-28ca-4497-a17f-97087cae7de9"
+          (reference "C801") (unit 1)
+        )
+      )
+    )
+  )
   (symbol (lib_id "Janelia:LED_DRIVER_LINEAR_BCR421U") (at 138.43 88.9 0) (unit 1)
