File: mouse-joystick-pcb/brake.kicad_sch (KiCad schematic)
At the start: 4 parts, among them J801 Conn_01x02_P3.5mm_TBH_Horizon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, U801 40V_200mA

Commit message: Update documentation for future v1.1
Other:
- company: Peter Polidoro -> Janelia Research Campus
Changed lines of the file:
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@@
 	(title_block
 		(title "mouse-joystick-pcb")
-		(date "2024-10-24")
-		(rev "1.0")
-		(company "Peter Polidoro")
+		(date "2026-01-15")
+		(rev "1.1")
+		(company "Janelia Research Campus")
+		(comment 1 "Peter Polidoro")
 	)
 	(text "30 Ohm ~ 40 mA ~ 2.6 newton-cm"
@@
 		(at 138.43 88.9 0)
 		(unit 1)
-		(exclude_from_sim yes)
+		(exclude_from_sim no)
 		(in_bom yes)
 		(on_board yes)
@@
 		(at 207.01 88.9 180)
 		(unit 1)
-		(exclude_from_sim yes)
+		(exclude_from_sim no)
 		(in_bom yes)
 		(on_board yes)
