File: mouse-joystick-pcb/motor-1.kicad_sch (KiCad schematic)
At the start: 21 parts, among them J701 Conn_01x02_P3.5mm_TBH_Horizon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, J702 Conn_01x04_P3.5mm_TBH_Horizon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, U701 MAX6816, U702 TMC5130A-TA, X701 16MHz_3.3V

Commit message: Finish routing
Parts:
- added R704: 1.8k, Janelia:R_0402_1005Metric, symbol Janelia:R_1.8k_0402
- C707: LCSC C2182652 -> C6119904; Manufacturer TDK Corporation -> HRE; Manufacturer Part Number C2012X5R1A476M125AC -> CGA0805X5R476M100MT; Vendor Digi-Key -> JLCPCB; Vendor Part Number 445-8239-1-ND -> C6119904
Connections:
- net VIO: now also R704.1
- net ~{CS}: now also R704.2
Changed lines of the file:
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@@
   (title_block
     (title "mouse-joystick-pcb")
-    (date "2024-10-15")
+    (date "2024-10-23")
     (rev "1.0")
     (company "Peter Polidoro")
@@
   (no_connect (at 36.83 124.46))
   (no_connect (at 36.83 127))
+  (wire (pts (xy 53.34 44.45) (xy 55.88 44.45))
+    (stroke (width 0) (type default))
+  )
   (wire (pts (xy 199.39 49.53) (xy 199.39 52.07))
     (stroke (width 0) (type default))
@@
     (stroke (width 0) (type default))
   )
+  (wire (pts (xy 95.25 86.36) (xy 95.25 88.9))
+    (stroke (width 0) (type default))
+  )
   (wire (pts (xy 62.23 68.58) (xy 62.23 66.04))
     (stroke (width 0) (type default))
@@
     (stroke (width 0) (type default))
   )
+  (wire (pts (xy 95.25 73.66) (xy 95.25 71.12))
+    (stroke (width 0) (type default))
+  )
   (wire (pts (xy 36.83 88.9) (xy 34.29 88.9))
     (stroke (width 0) (type default))
@@
     (effects (font (size 1.27 1.27)) (justify right bottom))
   )
+  (label "VIO" (at 95.25 71.12 90) (fields_autoplaced)
+    (effects (font (size 1.27 1.27)) (justify left bottom))
+  )
   (label "REFL" (at 40.64 177.8 180) (fields_autoplaced)
     (effects (font (size 1.27 1.27)) (justify right bottom))
   )
+  (label "~{CS}" (at 95.25 88.9 270) (fields_autoplaced)
+    (effects (font (size 1.27 1.27)) (justify right bottom))
+  )
   (label "GND" (at 34.29 111.76 180) (fields_autoplaced)
     (effects (font (size 1.27 1.27)) (justify right bottom))
@@
     (effects (font (size 1.27 1.27)) (justify right bottom))
   )
+  (label "~{CS}" (at 34.29 86.36 180) (fields_autoplaced)
+    (effects (font (size 1.27 1.27)) (justify right bottom))
+  )
   (label "BMA2" (at 74.93 86.36 0) (fields_autoplaced)
     (effects (font (size 1.27 1.27)) (justify left bottom))
@@
     (effects (font (size 1.27 1.27)) (justify right bottom))
   )
+  (label "~{CS}" (at 55.88 44.45 0) (fields_autoplaced)
+    (effects (font (size 1.27 1.27)) (justify left bottom))
+  )
   (label "GND" (at 199.39 78.74 270) (fields_autoplaced)
     (effects (font (size 1.27 1.27)) (justify right bottom))
@@
     (effects (font (size 1.27 1.27)) (justify left bottom))
   )
-  (hierarchical_label "~{CS}" (shape input) (at 34.29 86.36 180) (fields_autoplaced)
+  (hierarchical_label "COPI" (shape input) (at 34.29 91.44 180) (fields_autoplaced)
     (effects (font (size 1.27 1.27)) (justify right))
   )
-  (hierarchical_label "COPI" (shape input) (at 34.29 91.44 180) (fields_autoplaced)
+  (hierarchical_label "~{CS}" (shape input) (at 53.34 44.45 180) (fields_autoplaced)
     (effects (font (size 1.27 1.27)) (justify right))
   )
@@
       (effects (font (size 1.524 1.524)))
     )
-    (property "Vendor" "Digi-Key" (at 189.23 39.37 0)
-      (effects (font (size 1.524 1.524)) hide)
-    )
-    (property "Vendor Part Number" "445-8239-1-ND" (at 191.77 36.83 0)
+    (property "Vendor" "JLCPCB" (at 189.23 39.37 0)
+      (effects (font (size 1.524 1.524)) hide)
+    )
+    (property "Vendor Part Number" "C6119904" (at 191.77 36.83 0)
       (effects (font (size 1.524 1.524)) hide)
     )
@@
       (effects (font (size 1.27 1.27)) hide)
     )
-    (property "Manufacturer" "TDK Corporation" (at 186.69 44.45 0)
-      (effects (font (size 1.27 1.27)) hide)
-    )
-    (property "Manufacturer Part Number" "C2012X5R1A476M125AC" (at 186.69 44.45 0)
+    (property "Manufacturer" "HRE" (at 186.69 44.45 0)
+      (effects (font (size 1.27 1.27)) hide)
+    )
+    (property "Manufacturer Part Number" "CGA0805X5R476M100MT" (at 186.69 44.45 0)
       (effects (font (size 1.27 1.27)) hide)
     )
@@
       (effects (font (size 1.524 1.524)) hide)
     )
-    (property "LCSC" "C2182652" (at 186.69 44.45 0)
+    (property "LCSC" "C6119904" (at 186.69 44.45 0)
       (effects (font (size 1.27 1.27)) hide)
     )
@@
         )
       )
+    )
+  )
+  (symbol (lib_id "Janelia:R_1.8k_0402") (at 95.25 80.01 0) (unit 1)
+    (in_bom yes) (on_board yes) (dnp no)
+    (property "Reference" "R704" (at 96.52 80.01 0)
+      (effects (font (size 1.016 1.016)) (justify left))
+    )
+    (property "Value" "1.8k" (at 95.25 80.01 90) (do_not_autoplace)
+      (effects (font (size 0.762 0.762)))
+    )
+    (property "Footprint" "Janelia:R_0402_1005Metric" (at 93.472 80.01 90)
+      (effects (font (size 0.762 0.762)) hide)
+    )
+    (property "Datasheet" "" (at 97.282 80.01 90)
+      (effects (font (size 0.762 0.762)))
+    )
+    (property "Vendor" "JLCPCB" (at 99.822 77.47 90)
+      (effects (font (size 1.524 1.524)) hide)
+    )
+    (property "Vendor Part Number" "C409855" (at 102.362 74.93 90)
+      (effects (font (size 1.524 1.524)) hide)
+    )
+    (property "Synopsis" "RES SMD 1.8K OHM 5% 100mW" (at 104.902 72.39 90)
+      (effects (font (size 1.524 1.524)) hide)
+    )
+    (property "Package" "0402" (at 95.25 80.01 0)
+      (effects (font (size 1.27 1.27)) hide)
+    )
+    (property "Manufacturer" "PANASONIC" (at 95.25 80.01 0)
+      (effects (font (size 1.27 1.27)) hide)
+    )
+    (property "Manufacturer Part Number" "ERJ2GEJ182X" (at 95.25 80.01 0)
+      (effects (font (size 1.27 1.27)) hide)
+    )
+    (property "LCSC" "C409855" (at 95.25 80.01 0)
+      (effects (font (size 1.27 1.27)) hide)
+    )
+    (pin "2")
+    (pin "1")
+    (instances
+      (project "mouse-joystick-pcb"
+        (path "/df2b2e89-e055-4140-95de-f1df723db034/2a7fc1c1-17fb-44db-bbed-eea6ab177680"
+          (reference "R704") (unit 1)
+        )
+      )
