File: mouse-joystick-pcb/audio.kicad_sch (KiCad schematic)
At the start: 8 parts, among them U4 TPA6204A1DRBR

Commit message: Adjust schmatic
Parts:
- renumbered C19 to C601, C20 to C602, C21 to C603, C22 to C604, R7 to R601, R8 to R602, SP1 to SP601, U4 to U601
Changed lines of the file:
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@@
   (symbol (lib_id "Janelia:R_40k_100mW_0603") (at 93.98 90.17 90) (unit 1)
     (in_bom yes) (on_board yes) (dnp no)
-    (property "Reference" "R7" (at 93.98 87.63 90)
+    (property "Reference" "R601" (at 93.98 87.63 90)
       (effects (font (size 1.016 1.016)))
     )
@@
       (project "mouse-joystick-pcb"
         (path "/df2b2e89-e055-4140-95de-f1df723db034/3ad4effc-6f5c-46f5-ab22-93378768066e"
-          (reference "R7") (unit 1)
+          (reference "R601") (unit 1)
         )
       )
@@
   (symbol (lib_id "Janelia:Amplifier_Audio_TPA6204A1DRBR") (at 148.59 95.25 0) (unit 1)
     (in_bom yes) (on_board yes) (dnp no) (fields_autoplaced)
-    (property "Reference" "U4" (at 163.83 83.82 0) (do_not_autoplace)
+    (property "Reference" "U601" (at 163.83 83.82 0) (do_not_autoplace)
       (effects (font (size 1.524 1.524)))
     )
@@
       (project "mouse-joystick-pcb"
         (path "/df2b2e89-e055-4140-95de-f1df723db034/3ad4effc-6f5c-46f5-ab22-93378768066e"
-          (reference "U4") (unit 1)
+          (reference "U601") (unit 1)
         )
       )
@@
   (symbol (lib_id "Janelia:C_0.22uF_25V_0402") (at 80.01 90.17 90) (unit 1)
     (in_bom yes) (on_board yes) (dnp no) (fields_autoplaced)
-    (property "Reference" "C19" (at 80.01 83.82 90)
+    (property "Reference" "C601" (at 80.01 83.82 90)
       (effects (font (size 1.016 1.016)))
     )
@@
       (project "mouse-joystick-pcb"
         (path "/df2b2e89-e055-4140-95de-f1df723db034/3ad4effc-6f5c-46f5-ab22-93378768066e"
-          (reference "C19") (unit 1)
+          (reference "C601") (unit 1)
         )
       )
@@
   (symbol (lib_id "Janelia:C_0.22uF_25V_0402") (at 85.09 104.14 180) (unit 1)
     (in_bom yes) (on_board yes) (dnp no) (fields_autoplaced)
-    (property "Reference" "C20" (at 88.9 103.505 0)
+    (property "Reference" "C602" (at 88.9 103.505 0)
       (effects (font (size 1.016 1.016)) (justify right))
     )
@@
       (project "mouse-joystick-pcb"
         (path "/df2b2e89-e055-4140-95de-f1df723db034/3ad4effc-6f5c-46f5-ab22-93378768066e"
-          (reference "C20") (unit 1)
+          (reference "C602") (unit 1)
         )
       )
@@
   (symbol (lib_id "Janelia:R_40k_100mW_0603") (at 93.98 96.52 90) (unit 1)
     (in_bom yes) (on_board yes) (dnp no)
-    (property "Reference" "R8" (at 93.98 93.98 90)
+    (property "Reference" "R602" (at 93.98 93.98 90)
       (effects (font (size 1.016 1.016)))
     )
@@
       (project "mouse-joystick-pcb"
         (path "/df2b2e89-e055-4140-95de-f1df723db034/3ad4effc-6f5c-46f5-ab22-93378768066e"
-          (reference "R8") (unit 1)
+          (reference "R602") (unit 1)
         )
       )
@@
   (symbol (lib_id "Janelia:Speaker_13x13mm_8Ohm_700mW") (at 214.63 93.98 0) (unit 1)
     (in_bom yes) (on_board yes) (dnp no) (fields_autoplaced)
-    (property "Reference" "SP1" (at 218.44 95.25 0) (do_not_autoplace)
+    (property "Reference" "SP601" (at 218.44 95.25 0) (do_not_autoplace)
       (effects (font (size 1.27 1.27)) (justify left))
     )
@@
       (project "mouse-joystick-pcb"
         (path "/df2b2e89-e055-4140-95de-f1df723db034/3ad4effc-6f5c-46f5-ab22-93378768066e"
-          (reference "SP1") (unit 1)
+          (reference "SP601") (unit 1)
         )
       )
@@
   (symbol (lib_id "Janelia:C_0.22uF_25V_0402") (at 132.08 124.46 180) (unit 1)
     (in_bom yes) (on_board yes) (dnp no) (fields_autoplaced)
-    (property "Reference" "C22" (at 135.89 123.825 0)
+    (property "Reference" "C604" (at 135.89 123.825 0)
       (effects (font (size 1.016 1.016)) (justify right))
     )
@@
       (project "mouse-joystick-pcb"
         (path "/df2b2e89-e055-4140-95de-f1df723db034/3ad4effc-6f5c-46f5-ab22-93378768066e"
-          (reference "C22") (unit 1)
+          (reference "C604") (unit 1)
         )
       )
@@
   (symbol (lib_id "Janelia:C_1uF_35V_0402") (at 132.08 66.04 0) (unit 1)
     (in_bom yes) (on_board yes) (dnp no)
-    (property "Reference" "C21" (at 134.62 64.77 0)
+    (property "Reference" "C603" (at 134.62 64.77 0)
       (effects (font (size 1.016 1.016)) (justify left))
     )
@@
       (project "mouse-joystick-pcb"
         (path "/df2b2e89-e055-4140-95de-f1df723db034/3ad4effc-6f5c-46f5-ab22-93378768066e"
-          (reference "C21") (unit 1)
-        )
-      )
+          (reference "C603") (unit 1)
+        )
+      )

Commit message: Update date
Other:
- company: (none) -> Peter Polidoro
- title: (none) -> mouse-joystick-pcb
Changed lines of the file:
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@@
 (kicad_sch (version 20230121) (generator eeschema)
   (paper "A4")
+  (title_block
+    (title "mouse-joystick-pcb")
+    (date "2024-10-07")
+    (rev "1.0")
+    (company "Peter Polidoro")
+  )
   (wire (pts (xy 90.17 53.34) (xy 92.71 53.34))
     (stroke (width 0) (type default))
