File: mouse-joystick-pcb/torque-sensor.kicad_sch (KiCad schematic)
At the start: 0 parts

Commit message: Add torque-sensor sheet
Parts:
- added C901, C902, C903, C904: 0.1uF_100V, Janelia:C_0402_1005Metric, symbol Janelia:C_0.1uF_100V_0402
- added J901: Conn_01x04_P3.5mm_TBH_Horizontal_Screw, Janelia:PhoenixContact_MC_1,5_4-G-3.5_1x04_P3.50mm_Horizontal_Screw, symbol Janelia:Conn_01x04_P3.5mm_TBH_Horizontal_Screw
- added U901: PGA305ARHHR, Janelia:RHH0036C, symbol Janelia:PGA305ARHHR
Connections:
- new net AVDD: C903.1, U901.9 (AVDD)
- new net BRG+: J901.1 (Pin_1), U901.15 (BRG+)
- new net BRG-: J901.4 (Pin_4), U901.14 (BRG-)
- new net DVDD: C902.1, U901.3 (DVDD)
- new net GND: C901.2, C902.2, C903.2, C904.2, U901.10 (GND), U901.23 (AVSS), U901.29 (I2CADDR), U901.32 (DVSS), U901.37 (PAD)
- new net INP+: J901.3 (Pin_3), U901.18 (INP+)
- new net INP-: J901.2 (Pin_2), U901.17 (INP-)
- new net REFCAP: C904.1, U901.16 (REFCAP)
- new net SCL: U901.36 (SCL)
- new net SDA: U901.33 (SDA)
- new net VPWR: C901.1, U901.5 (PWR)
- no-connect marks 0 -> 8
Other:
- note added: "BLACK"
- note added: "GREEN"
- note added: "I2CADDR - Logic 0 0x40, 0x42, 0x45"
- note added: "RED"
- note added: "WHITE"

Commit message: Complete some routing
Connections:
- net BRG+: now also J901.2 (Pin_2); no longer J901.1 (Pin_1)
- net BRG-: now also J901.1 (Pin_1); no longer J901.4 (Pin_4)
- net INP+: now also J901.4 (Pin_4); no longer J901.3 (Pin_3)
- net INP-: now also J901.3 (Pin_3); no longer J901.2 (Pin_2)
Other:
- company: (none) -> Peter Polidoro
- title: (none) -> mouse-joystick-pcb
Changed lines of the file:
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@@
 (kicad_sch (version 20230121) (generator eeschema)
   (paper "A4")
+  (title_block
+    (title "mouse-joystick-pcb")
+    (date "2024-10-15")
+    (rev "1.0")
+    (company "Peter Polidoro")
+  )
   (no_connect (at 140.97 83.82))
   (no_connect (at 140.97 99.06))
@@
     (stroke (width 0) (type default))
   )
-  (text "GREEN" (at 198.12 90.17 0)
-    (effects (font (size 1.27 1.27)) (justify right bottom))
-  )
-  (text "BLACK" (at 198.12 87.63 0)
-    (effects (font (size 1.27 1.27)) (justify right bottom))
-  )
-  (text "RED" (at 198.12 95.25 0)
+  (text "GREEN" (at 198.12 87.63 0)
+    (effects (font (size 1.27 1.27)) (justify right bottom))
+  )
+  (text "BLACK" (at 198.12 95.25 0)
+    (effects (font (size 1.27 1.27)) (justify right bottom))
+  )
+  (text "RED" (at 198.12 92.71 0)
     (effects (font (size 1.27 1.27)) (justify right bottom))
   )
@@
     (effects (font (size 1.27 1.27)) (justify right bottom))
   )
-  (text "WHITE" (at 198.12 92.71 0)
+  (text "WHITE" (at 198.12 90.17 0)
     (effects (font (size 1.27 1.27)) (justify right bottom))
   )
@@
     (effects (font (size 1.27 1.27)) (justify right bottom))
   )
-  (label "BRG-" (at 204.47 87.63 180) (fields_autoplaced)
+  (label "BRG-" (at 204.47 95.25 180) (fields_autoplaced)
     (effects (font (size 1.27 1.27)) (justify right bottom))
   )
@@
     (effects (font (size 1.27 1.27)) (justify right bottom))
   )
-  (label "INP-" (at 204.47 92.71 180) (fields_autoplaced)
+  (label "INP-" (at 204.47 90.17 180) (fields_autoplaced)
     (effects (font (size 1.27 1.27)) (justify right bottom))
   )
@@
     (effects (font (size 1.27 1.27)) (justify left bottom))
   )
-  (label "INP+" (at 204.47 90.17 180) (fields_autoplaced)
-    (effects (font (size 1.27 1.27)) (justify right bottom))
-  )
-  (label "BRG+" (at 204.47 95.25 180) (fields_autoplaced)
+  (label "INP+" (at 204.47 87.63 180) (fields_autoplaced)
+    (effects (font (size 1.27 1.27)) (justify right bottom))
+  )
+  (label "BRG+" (at 204.47 92.71 180) (fields_autoplaced)
     (effects (font (size 1.27 1.27)) (justify right bottom))
   )
@@
   )
   (symbol (lib_id "Janelia:PGA305ARHHR") (at 118.11 91.44 0) (unit 1)
-    (in_bom yes) (on_board yes) (dnp no) (fields_autoplaced)
+    (in_bom yes) (on_board yes) (dnp no)
     (property "Reference" "U901" (at 133.35 73.66 0) (do_not_autoplace)
       (effects (font (size 1.524 1.524)))
     )
-    (property "Value" "PGA305ARHHR" (at 118.11 91.44 0) (do_not_autoplace)
+    (property "Value" "PGA305ARHHR" (at 100.33 73.66 0) (do_not_autoplace)
       (effects (font (size 1.524 1.524)))
     )
@@
       (effects (font (size 1.27 1.27)) hide)
     )
-    (property "Sim.Enable" "0" (at 118.11 91.44 0)
-      (effects (font (size 1.27 1.27)) hide)
-    )
-    (property "LCSC" "C2678416" (at 118.11 91.44 0)
-      (effects (font (size 1.27 1.27)) hide)
-    )
+    (property "Sim.Enable" "0" (at 118.11 38.1 0)
+      (effects (font (size 1.27 1.27)) hide)
+    )
+    (property "LCSC" "C2678416" (at 118.11 58.42 0)
+      (effects (font (size 1.27 1.27)) hide)
+    )

Commit message: Finish routing
Other:
- note removed: "BLACK"
- note removed: "GREEN"
- note removed: "RED"
- note removed: "WHITE"
Changed lines of the file:
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@@
   (title_block
     (title "mouse-joystick-pcb")
-    (date "2024-10-15")
+    (date "2024-10-23")
     (rev "1.0")
     (company "Peter Polidoro")
@@
     (stroke (width 0) (type default))
   )
-  (text "GREEN" (at 198.12 87.63 0)
-    (effects (font (size 1.27 1.27)) (justify right bottom))
-  )
-  (text "BLACK" (at 198.12 95.25 0)
-    (effects (font (size 1.27 1.27)) (justify right bottom))
-  )
-  (text "RED" (at 198.12 92.71 0)
-    (effects (font (size 1.27 1.27)) (justify right bottom))
-  )
   (text "I2CADDR - Logic 0\n0x40, 0x42, 0x45" (at 83.82 87.63 0)
     (effects (font (size 1.27 1.27)) (justify right bottom))
   )
-  (text "WHITE" (at 198.12 90.17 0)
-    (effects (font (size 1.27 1.27)) (justify right bottom))
-  )
