File: mouse-joystick-pcb/torque-sensor.kicad_sch (KiCad schematic)
At the start: 6 parts, among them J901 Conn_01x04_P3.5mm_TBH_Horizon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, U901 PGA305ARHHR

Commit message: Update documentation for future v1.1
Other:
- company: Peter Polidoro -> Janelia Research Campus
Changed lines of the file:
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@@
 	(title_block
 		(title "mouse-joystick-pcb")
-		(date "2024-10-24")
-		(rev "1.0")
-		(company "Peter Polidoro")
+		(date "2026-01-15")
+		(rev "1.1")
+		(company "Janelia Research Campus")
+		(comment 1 "Peter Polidoro")
 	)
 	(text "I2CADDR - Logic 0\n0x40, 0x42, 0x45"
@@
 		(at 118.11 91.44 0)
 		(unit 1)
-		(exclude_from_sim yes)
+		(exclude_from_sim no)
 		(in_bom yes)
 		(on_board yes)
@@
 		(at 212.09 92.71 180)
 		(unit 1)
-		(exclude_from_sim yes)
+		(exclude_from_sim no)
 		(in_bom yes)
 		(on_board yes)
