File: mouse-joystick-pcb/base-motor.kicad_sch (KiCad schematic)
At the start: 22 parts, among them J701 Conn_01x02_P3.5mm_TBH_Horizon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, J702 Conn_01x04_P3.5mm_TBH_Horizon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, U701 MAX6816, U702 TMC5130A-TA, X701 16MHz_3.3V

Commit message: Update documentation for future v1.1
Other:
- company: Peter Polidoro -> Janelia Research Campus
Changed lines of the file:
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@@
 	(title_block
 		(title "mouse-joystick-pcb")
-		(date "2024-10-24")
-		(rev "1.0")
-		(company "Peter Polidoro")
+		(date "2026-01-15")
+		(rev "1.1")
+		(company "Janelia Research Campus")
+		(comment 1 "Peter Polidoro")
 	)
 	(text "1.64 A RMS\n"
@@
 		(at 124.46 101.6 180)
 		(unit 1)
-		(exclude_from_sim yes)
+		(exclude_from_sim no)
 		(in_bom yes)
 		(on_board yes)
@@
 		(at 53.34 176.53 0)
 		(unit 1)
-		(exclude_from_sim yes)
+		(exclude_from_sim no)
 		(in_bom yes)
 		(on_board yes)
@@
 		(at 100.33 179.07 180)
 		(unit 1)
-		(exclude_from_sim yes)
+		(exclude_from_sim no)
 		(in_bom yes)
 		(on_board yes)
